File: hardware/pcb_design/Custom_board.kicad_pcb (KiCad board)
At the start: 2 copper layers, 6 parts, among them J1 Rpi, U1 ESP32-DEVKIT-V1, U3 ROB-14450

Commit message: Add files via upload
PCB design updated
Parts:
- added J2: Conn_01x02, Connector_PinSocket_2.54mm:PinSocket_1x02_P2.54mm_Vertical, F.Cu at (183.0, 94.8)
- added J3: Conn_01x02, Connector_PinSocket_2.54mm:PinSocket_1x02_P2.54mm_Vertical, F.Cu at (183.0, 115.5)
- added J4: Conn_01x01, Connector_PinSocket_2.54mm:PinSocket_1x01_P2.54mm_Vertical, F.Cu at (200.3, 100.3)
- added J5: Conn_01x01, Connector_PinSocket_2.54mm:PinSocket_1x01_P2.54mm_Vertical, F.Cu at (244.5, 111.5)
- moved J1 120.3 mm to (242.7, 91.0), turned to 0 degrees
- moved MPU6050 88.4 mm to (211.7, 69.5), turned to 90 degrees
- moved U1 80.2 mm to (224.5, 101.5), turned to 180 degrees
- moved MOTOR_B1 74.8 mm to (198.5, 124.0), turned to 180 degrees
- moved MOTOR_A1 63.6 mm to (198.5, 80.3)
- moved U3 26.6 mm to (197.6, 101.8), turned to 0 degrees
Connections:
- MOTOR_A1 pad 6: +3V3 -> /V
- MOTOR_B1 pad 6: +3V3 -> /V
- MPU6050 pad 1: +3V3 -> /V
- U1 pad 1: +3V3 -> /V
- U1 pad 10: /ENCA_B -> unconnected-(U1-D19-Pad10)
- U1 pad 15: unconnected-(U1-D23-Pad15) -> /15
- U1 pad 16: +3V3 -> unconnected-(U1-EN-Pad16)
- U1 pad 19: /ENCB_A -> /ENCA_B
- U1 pad 20: /ENCB_B -> /ENCA_A
- U1 pad 21: /32 -> /21
- U1 pad 22: /33 -> /22
- U1 pad 23: /25 -> /23
- U1 pad 24: /26 -> /24
- U1 pad 25: /27 -> /25
- U1 pad 26: /14 -> /26
- U1 pad 27: unconnected-(U1-D12-Pad27) -> /ENCB_A
- U1 pad 28: unconnected-(U1-D13-Pad28) -> /ENCB_B
- U1 pad 9: /ENCA_A -> unconnected-(U1-D18-Pad9)
- U3 pad 10: /32 -> /26
- U3 pad 11: /33 -> /25
- U3 pad 12: /25 -> /24
- U3 pad 13: +3V3 -> /V
- U3 pad 14: /27 -> /23
- U3 pad 15: /26 -> /22
- U3 pad 16: /14 -> /21
Routing:
- net +3V3: track 188.6 -> 0.00 mm
- net /V: track 0.00 -> 126.7 mm
- net /ENCB_B: track 61.3 -> 17.3 mm
- net /A+: track 73.2 -> 32.5 mm
- net GND: track 216.8 -> 176.8 mm
- net /ENCA_B: track 54.0 -> 15.9 mm
- net /ENCB_A: track 56.0 -> 18.4 mm
- net /14: track 37.4 -> 0.00 mm
- net /5V: track 33.1 -> 67.2 mm
- net /27: track 33.2 -> 0.00 mm
- net /ENCA_A: track 47.7 -> 16.4 mm
- net /A-: track 55.6 -> 26.8 mm
- net /33: track 27.4 -> 0.00 mm
- net /26: track 33.2 -> 7.14 mm
- net /25: track 30.2 -> 7.14 mm
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- added copper zone on F.Cu, net (none)
- added copper zone on F.Cu, net GND
Other:
- board outline added: 70 x 66.5 mm
- board text added: "+"
- board text added: "-"
- board text added: "12V"
- board text added: "5V"
