File: hardware/pcb_design/Custom_board.kicad_sch (KiCad schematic)
At the start: 6 parts, among them J1 Rpi, U1 ESP32-DEVKIT-V1, U3 ROB-14450

Commit message: Add files via upload
PCB design updated
Parts:
- added J2, J3: Conn_01x02, Connector_PinSocket_2.54mm:PinSocket_1x02_P2.54mm_Vertical, symbol Connector_Generic:Conn_01x02
- added J4, J5: Conn_01x01, Connector_PinSocket_2.54mm:PinSocket_1x01_P2.54mm_Vertical, symbol Connector_Generic:Conn_01x01
Connections:
- net +12V: now also J2.1 (Pin_1)
- net 25: now also U1.25 (D27), U3.11 (BI2); no longer U1.23 (D25), U3.12 (BI1)
- net 26: now also U1.26 (D14), U3.10 (PWMB); no longer U1.24 (D26), U3.15 (AI2)
- net 5V: now also J3.1 (Pin_1)
- net ENCA_A: now also U1.20 (D35); no longer U1.9 (D18)
- net ENCA_B: now also U1.19 (D34); no longer U1.10 (D19)
- net ENCB_A: now also U1.27 (D12); no longer U1.19 (D34)
- net ENCB_B: now also U1.28 (D13); no longer U1.20 (D35)
- net GND: now also J2.2 (Pin_2), J3.2 (Pin_2)
- net 15: now reaches U1.15 (D23)
- net +3V3 renamed V
- net V: now also J4.1 (Pin_1), J5.1 (Pin_1); no longer U1.16 (EN)
- net 14 renamed 21
- net 21: now also U1.21 (D32); no longer U1.26 (D14)
- net 27 renamed 23
- net 23: now also U1.23 (D25); no longer U1.25 (D27)
- removed net 32: U1.21 (D32), U3.10 (PWMB)
- net 33 renamed 22
- net 22: now also U3.15 (AI2); no longer U3.11 (BI2)
- new net 24: U1.24 (D26), U3.12 (BI1)
- no-connect marks 0 -> 13
Other:
- moved on the sheet: MOTOR_A1, MPU6050
